File: CANbus_Logging_Bridge/CANbus_Logging_Bridge.kicad_pcb (KiCad board)
At the start: 4 copper layers, 110 x 141 mm, 254 parts, among them J1 USB_C_Receptacle, J10 Conn_02x02_Pin, J11 Conn_01x08_Socket, J12 Conn_01x08_Socket, J13 Conn_01x08_Socket, J14 Conn_01x08_Socket, J15 Conn_01x08_Socket, J16 Conn_01x08_Socket, J2 Screw_Terminal_01x02, J3 FPS009-4200-0, J4 Conn_02x03_Odd_Even, J5 Conn_02x02_Pin, J6 Conn_02x02_Pin, J7 Conn_02x02_Pin, J8 Conn_02x02_Pin, J9 Conn_02x02_Pin, SW1 SMD_5.2x5.2mm_h1.9mm, SW2 SMD_5.2x5.2mm_h1.9mm, U1 RV-3028-C7, U10 MCP2515-xSO, U11 MCP2515-xSO, U12 MCP2515-xSO, U13 MCP2515-xSO, U14 ISOW1044, U15 ISOW1044, U16 ISOW1044, U17 ISOW1044, U18 ISOW1044, U19 ISOW1044, U2 ESP32-S3-WROOM, U3 LM1085-3.3, U4 LM1085-5.0, U5 AP2112K-3.3, U6 TCA9534, U7 TCA9534, U8 MCP2515-xSO, U9 MCP2515-xSO, Y1 20MHz, Y2 20MHz, Y3 20MHz, Y4 20MHz, Y5 20MHz, Y6 20MHz

Commit message: Layout v01
-Add Silk
-Ground Stitching
Parts:
- added G***: LOGO, Logging_Bridge_Lib:QR, B.Cu at (55.5, 158.5)
- added REF**: Standoff, Logging_Bridge_Lib:Standoff, F.Cu at (94.0, 37.0)
- added kibuzzard-683381FB: G***, kibuzzard-683381FB, F.Cu at (54.0, 42.0)
- added kibuzzard-68338202: G***, kibuzzard-68338202, F.Cu at (70.7, 42.0)
- added kibuzzard-6833820A: G***, kibuzzard-6833820A, F.Cu at (42.5, 60.5)
- added kibuzzard-683384E4: G***, kibuzzard-683384E4, F.Cu at (48.5, 105.5)
- added kibuzzard-683384F2: G***, kibuzzard-683384F2, F.Cu at (48.0, 121.5)
- added kibuzzard-6833851A: G***, kibuzzard-6833851A, F.Cu at (49.5, 93.4)
- added kibuzzard-6833856B: G***, kibuzzard-6833856B, F.Cu at (105.5, 41.4)
- added kibuzzard-6833858D: G***, kibuzzard-6833858D, F.Cu at (105.5, 62.8)
- added kibuzzard-68338593: G***, kibuzzard-68338593, F.Cu at (105.5, 84.6)
- added kibuzzard-6833859C: G***, kibuzzard-6833859C, F.Cu at (105.5, 105.7)
- added kibuzzard-683385A1: G***, kibuzzard-683385A1, F.Cu at (105.5, 127.8)
- added kibuzzard-683385A6: G***, kibuzzard-683385A6, F.Cu at (105.5, 149.4)
- added kibuzzard-68338682: G***, kibuzzard-68338682, F.Cu at (114.0, 37.0)
- added kibuzzard-68339090: G***, kibuzzard-68339090, F.Cu at (48.0, 81.5)
- added kibuzzard-683390BD: G***, kibuzzard-683390BD, F.Cu at (52.0, 81.5)
- added kibuzzard-683390C2: G***, kibuzzard-683390C2, F.Cu at (52.0, 84.0)
- added kibuzzard-683390DA: G***, kibuzzard-683390DA, F.Cu at (52.0, 86.5)
- added kibuzzard-683390E1: G***, kibuzzard-683390E1, F.Cu at (48.0, 86.5)
- added kibuzzard-683390E7: G***, kibuzzard-683390E7, F.Cu at (48.0, 84.0)
- added kibuzzard-68339145: G***, kibuzzard-68339145, F.Cu at (86.0, 74.5)
- added kibuzzard-6833916E: G***, kibuzzard-6833916E, F.Cu at (66.0, 105.0)
- added kibuzzard-6833918D: G***, kibuzzard-6833918D, F.Cu at (83.0, 141.0)
- added kibuzzard-68339228: G***, kibuzzard-68339228, F.Cu at (135.0, 173.5)
- added kibuzzard-683393CD: G***, kibuzzard-683393CD, B.Cu at (55.5, 141.0)
- added kibuzzard-68339419: G***, kibuzzard-68339419, F.Cu at (145.0, 121.5)
- added kibuzzard-68339449: G***, kibuzzard-68339449, F.Cu at (145.0, 124.0)
- added kibuzzard-68339454: G***, kibuzzard-68339454, F.Cu at (145.5, 111.5)
- added kibuzzard-6833959C: G***, kibuzzard-6833959C, F.Cu at (137.7, 52.0)
- moved REF** 4.96 mm to (94.0, 172.0)
- moved U7 4.19 mm to (82.8, 147.8)
- moved R21 4.19 mm to (84.0, 154.5)
- moved D22 2.26 mm to (42.5, 62.6)
- moved R51 2.26 mm to (42.5, 65.5)
Routing:
- net 3.3V: track 475.6 -> 484.0 mm
- net Net-(D15-A): track 34.1 -> 38.3 mm
- net Net-(D14-A): track 15.7 -> 19.9 mm
- net Net-(D11-A): track 60.0 -> 64.2 mm
- net Net-(D10-A): track 79.0 -> 83.1 mm
- net SDA: track 149.4 -> 153.6 mm
- net SCL: track 152.6 -> 156.7 mm
- net Net-(D9-A): track 100.4 -> 104.6 mm
- net Net-(D8-A): track 118.4 -> 122.6 mm
- net VIN: track 72.2 -> 74.5 mm
- net Net-(D12-A): track 56.1 -> 57.8 mm
- net Net-(D13-A): track 53.5 -> 55.2 mm
- net ISOGND6: vias 4 -> 28
- net ISOGND5: vias 4 -> 28
- net ISOGND4: vias 4 -> 28
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