File: CANbus_Logging_Bridge/CANbus_Logging_Bridge.kicad_sch (KiCad schematic)
At the start: 219 parts, among them J1 8P8C, J2 USB_C_Receptacle, J3 microSD_Friction, J4 8P8C, J5 8P8C, J6 8P8C, J7 8P8C, J8 8P8C, J9 Screw_Terminal_01x02, SW1 SMD_5.2x5.2mm_h1.9mm, SW2 SMD_5.2x5.2mm_h1.9mm, U1 ESP32-S3-WROOM, U10 MCP2515-xSO, U11 MCP2515-xSO, U12 MCP2515-xSO, U13 ISOW1044, U14 ISOW1044, U15 ISOW1044, U16 RV-1805-C3, U17 TCA9534, U18 TCA9534, U19 AP2112K-3.3, U2 MCP2515-xSO, U3 ISOW1044, U4 LM1085-3.3, U5 LM1085-5.0, U6 MCP2515-xSO, U7 ISOW1044, U8 MCP2515-xSO, U9 ISOW1044, Y1 20MHz, Y2 20MHz, Y3 20MHz, Y4 20MHz, Y5 20MHz, Y6 20MHz

Commit message: v01 layout pre-silk
Project:
-Add datasheets
SCH:
-Add termination resistors/jumpers to CAN lines
-Swap microSD socket to full SD socket
-Change RJ45 pinout to VE.Can pinout
-Double check SPI pinout on ESP32
-Reverse CAN ~{RST} bias so that devices are held in reset by default
-Move LED off IO0 and add 0.1 capacitor
-Address USB power situation
-Connect CAN ~{INT} lines to ESP32
-Breakout EN, IO0, U0TXD, U0RXD, 3.3V and GND
-Update RTC (Part is NRFND)
-Add Power Status LEDs
BRD:
-v01 layout
Parts:
- removed C85: 47pF, Logging_Bridge_Lib:C_0402_1005Metric, symbol Logging_Bridge_Lib:47pF_0402_500V_10%
- removed D19, D20: BAT60A, Logging_Bridge_Lib:SOD-323, symbol Logging_Bridge_Lib:D_Schottky_3A_10V_0.28V
- removed J1, J4, J5, J6, J7, J8: 8P8C, Logging_Bridge_Lib:RJ45_OST_PJ012-8P8CX_Vertical, symbol Logging_Bridge_Lib:8P8C
- removed J3: microSD_Friction, SparkFun-Connector:microSD_Friction_Fit_Common, symbol Logging_Bridge_Lib:microSD_Friction
- removed R15, R16, R2, R23, R24, R25: 10k, Logging_Bridge_Lib:R_0402_1005Metric, symbol Logging_Bridge_Lib:10k_0402
- removed U16: RV-1805-C3, Logging_Bridge_Lib:RTC_SMD_MicroCrystal_C3_2.5x3.7mm, symbol Logging_Bridge_Lib:RV-1805-C3
- added C3: 100nF, Logging_Bridge_Lib:C_0402_1005Metric, symbol Logging_Bridge_Lib:10nF_0402_25V_10%
- added C5: 0.1uF, Logging_Bridge_Lib:C_0402_1005Metric, symbol Logging_Bridge_Lib:0.1uF_0402_16V_10%
- added C92, C93, C94, C95, C96, C97: 4.7nF, Logging_Bridge_Lib:C_0402_1005Metric, symbol Logging_Bridge_Lib:4.7nF_0402
- added D22: Red, Logging_Bridge_Lib:LED_0603_1608Metric, symbol Logging_Bridge_Lib:LED_Red_0603
- added D3, D4, D5: SK34A, Logging_Bridge_Lib:SMA, symbol Logging_Bridge_Lib:D_Schottky_3A_40V_0.55V
- added J10, J5, J6, J7, J8, J9: Conn_02x02_Pin, Logging_Bridge_Lib:PinHeader_2x02_P2.54mm_Vertical_SMD, symbol Logging_Bridge_Lib:Conn_01x04_Pin
- added J11, J12, J13, J14, J15, J16: Conn_01x08_Socket, Logging_Bridge_Lib:1x08, symbol Logging_Bridge_Lib:Conn_01x08_Socket
- added J3: FPS009-4200-0, Logging_Bridge_Lib:FPS00942000, symbol Logging_Bridge_Lib:FPS009-4200-0
- added J4: Conn_02x03_Odd_Even, Logging_Bridge_Lib:PinHeader_2x03_P2.54mm_Vertical, symbol Logging_Bridge_Lib:Conn_02x03_Odd_Even
- added R10, R12, R6, R9: 10k, Logging_Bridge_Lib:R_0402_1005Metric, symbol Logging_Bridge_Lib:10k_0402
- added R39, R40, R41, R42, R43, R44, R45, R46, R47, R48, R49, R50: 60, Logging_Bridge_Lib:R_0402_1005Metric, symbol Logging_Bridge_Lib:60_0402_1
- added R51: 2.0k, Logging_Bridge_Lib:R_1206_3216Metric, symbol Logging_Bridge_Lib:2.0k_1206
- added TP1: 1.0mm, Logging_Bridge_Lib:TestPoint-1.0mm, symbol Logging_Bridge_Lib:TestPoint_1.0mm
- added U1: RV-3028-C7, Logging_Bridge_Lib:MicroCrystal_C7_SON-8_1.5x3.2mm_P0.9mm, symbol Logging_Bridge_Lib:RV-3028-C7
- C15: footprint Logging_Bridge_Lib:C_0402_1005Metric -> Logging_Bridge_Lib:C_0603_1608Metric
- C16: renamed from C18; footprint Logging_Bridge_Lib:C_0402_1005Metric -> Logging_Bridge_Lib:C_0603_1608Metric
- C2: renamed from C86; value 10nF -> 100nF; PROD_ID CAP-16508 -> (none)
- renumbered C84 to C1, C16 to C10, C90 to C11, C13 to C12, C17 to C13, C89 to C14, C88 to C17, C20 to C18, C21 to C19, C12 to C20, C19 to C21, C35 to C22, C47 to C23, C48 to C24, C49 to C25, C3 to C26, C4 to C27, C24 to C28, C25 to C29, C36 to C30, C37 to C31, C50 to C32, C51 to C33, C52 to C34, C53 to C35, C54 to C36, C55 to C37, C9 to C38, C26 to C39, C23 to C4, C38 to C40, C56 to C41, C57 to C42, C58 to C43, C10 to C44, C27 to C45, C39 to C46, C59 to C47, C60 to C48, C61 to C49, C6 to C50, C28 to C51, C40 to C52, C62 to C53, C63 to C54, C64 to C55, C11 to C56, C29 to C57, C41 to C58, C65 to C59, C83 to C6, C66 to C60, C67 to C61, C1 to C62, C8 to C63, C30 to C64, C31 to C65, C42 to C66, C43 to C67, C22 to C7, C7 to C74, C2 to C75, C32 to C76, C33 to C77, C44 to C78, C45 to C79, C87 to C8, C74 to C80, C75 to C81, C76 to C82, C77 to C83, C78 to C84, C79 to C85, C5 to C86, C34 to C87, C46 to C88, C80 to C89, C14 to C9, C81 to C90, C82 to C91, D8 to D1, D11 to D10, D12 to D11, D13 to D12, D14 to D13, D15 to D14, D16 to D15, D1 to D16, D3 to D17, D4 to D18, D5 to D19, D6 to D20, D7 to D21, D17 to D6, D18 to D7, D9 to D8, D10 to D9, J2 to J1, J9 to J2, L6 to L1, L19 to L10, L20 to L11, L21 to L12, L5 to L13, L8 to L14, L13 to L15, L22 to L16, L23 to L17, L24 to L18, L2 to L19, L3 to L2, L1 to L20, L9 to L21, L10 to L22, L14 to L23, L15 to L24, L7 to L3, L11 to L5, L12 to L6, L16 to L7, L17 to L8, L18 to L9, R28 to R1, R41 to R14, R40 to R15, R26 to R16, R6 to R17, R27 to R18, R7 to R19, R42 to R2, R8 to R20, R30 to R21, R5 to R22, R4 to R23, R3 to R24, R43 to R25, R44 to R26, R45 to R27, R46 to R28, R47 to R29, R9 to R3, R48 to R30, R49 to R31, R50 to R32, R1 to R33, R12 to R34, R14 to R35, R18 to R36, R19 to R37, R20 to R38, R10 to R4, R21 to R5, R29 to R7, R17 to R8, TP1 to TP2, TP2 to TP3, U8 to U10, U10 to U11, U11 to U12, U12 to U13, U3 to U14, U7 to U15, U9 to U16, U13 to U17, U14 to U18, U15 to U19, U1 to U2, U4 to U3, U5 to U4, U19 to U5, U17 to U6, U18 to U7, U2 to U8, U6 to U9
Connections:
- net 3.3V: now also C3.1, J3.4 (VDD), J4.2 (Pin_2), U1.7 (VDD); no longer R11.1, R13.1, R8.1
- net CS_CAN1: now also U2.34 (IO41); no longer U2.17 (IOA9)
- net CS_CAN2: now also U2.32 (IO39); no longer U2.18 (IOA10)
- net CS_CAN3: now also U2.24 (IO47); no longer U2.19 (IOA11)
- net CS_CAN4: now also U2.22 (IOA14); no longer U2.20 (IOA12)
- net CS_CAN5: now also U2.20 (IOA12); no longer U2.21 (IOA13)
- net CS_CAN6: now also U2.11 (IOA18); no longer U2.22 (IOA14)
- net ESP_STATUS: now also U2.31 (IO38); no longer SW2.2, U2.27 (IO0)
- net GND: now also C1.-, R11.2, R13.2, R8.2, C3.2, C5.1, D22.1 (K), J3.10 (SHIELD), J3.11 (SHIELD), J3.12 (SHIELD), J3.13 (SHIELD), J3.3 (VSS), J3.6 (VSS), J4.4 (Pin_4), R10.2, R12.2, R6.1, R9.2, U1.5 (VSS); no longer C1.2
- net ISOGND1: now also U14.16 (GISOIN), U14.17 (GISOIN), C92.2, J11.3 (Pin_3)
- net ISOGND2: now also U15.16 (GISOIN), U15.17 (GISOIN), C93.2, J12.3 (Pin_3)
- net ISOGND3: now also U16.16 (GISOIN), U16.17 (GISOIN), C94.2, J13.3 (Pin_3)
- net ISOGND4: now also U17.16 (GISOIN), U17.17 (GISOIN), C95.2, J14.3 (Pin_3)
- net ISOGND5: now also U18.16 (GISOIN), U18.17 (GISOIN), C96.2, J15.3 (Pin_3)
- net ISOGND6: now also U19.16 (GISOIN), U19.17 (GISOIN), C97.2, J16.3 (Pin_3)
- net PICO: now also U2.18 (IOA10); no longer U2.33 (IO40)
- net POCI: now also U2.17 (IOA9); no longer U2.32 (IO39)
- net RTC_BAT: now also U1.6 (VBACKUP)
- net SCK: now also U2.19 (IOA11); no longer U2.31 (IO38)
- net SCL: now also U2.38 (IOA2), U1.3 (SCL); no longer U2.35 (IO42)
- net SDA: now also U2.39 (IOA1), U1.4 (SDA); no longer U2.34 (IO41)
- net SD_CLK: now also J3.5 (CLK)
- net SD_CMD: now also J3.2 (CMD)
- net SD_DAT0: now also J3.7 (DAT0)
- net SD_DAT1: now also J3.8 (DAT1)
- net SD_DAT2: now also J3.9 (DAT2)
- net SD_DAT3: now also J3.1 (DAT3)
- net VIN: now also D3.A, D4.A, R51.2; no longer U3.3 (VI), U4.3 (VI)
- net VUSB: now also D5.A; no longer U5.1 (VIN)
- net ~{RST_CAN1}: now also R13.1, U6.10 (P5); no longer U6.4 (P0)
- net ~{RST_CAN2}: now also U6.9 (P4), R12.1; no longer R11.2, U6.5 (P1)
- net ~{RST_CAN3}: now also U6.5 (P1), R9.1; no longer R13.2, U6.6 (P2)
- net ~{RST_CAN4}: now also R8.1, U6.4 (P0); no longer U6.7 (P3)
- net ~{RST_CAN5}: now also R11.1, U6.7 (P3); no longer U6.9 (P4)
- net ~{RST_CAN6}: now also U6.6 (P2), R10.1; no longer R8.2, U6.10 (P5)
- net ~{INT_CAN6}: now reaches U13.12 (~{INT})
- net ~{INT_CAN6}: now also U2.12 (IOA8)
- net at D21.1 (A1), U19.18 (CANL): now also J10.2 (Pin_2), J16.8 (Pin_8)
- net at D21.2 (A2), U19.19 (CANH): now also J10.4 (Pin_4), J16.7 (Pin_7)
- net at D19.1 (A1), U17.18 (CANL): now also J14.8 (Pin_8), J8.2 (Pin_2)
- net at D19.2 (A2), U17.19 (CANH): now also J14.7 (Pin_7), J8.4 (Pin_4)
- net ~{INT_CAN4}: now reaches U11.12 (~{INT})
- net ~{INT_CAN4}: now also U2.23 (IO21)
- net CAN1_P: now reaches D16.2 (A2), U14.19 (CANH)
- net CAN1_P: now also J11.7 (Pin_7), J5.4 (Pin_4)
- net CAN1_N: now reaches D16.1 (A1), U14.18 (CANL)
- net CAN1_N: now also J11.8 (Pin_8), J5.2 (Pin_2)
- net ESP32_EN: now reaches C6.1, R5.1, SW1.2, U2.3 (EN)
- net ESP32_EN: now also J4.1 (Pin_1)
- net ~{INT_CAN3}: now reaches U10.12 (~{INT})
- net ~{INT_CAN3}: now also U2.25 (IO48)
- net ESP32_RXD: now reaches U2.36 (RXD0/IO44)
- net ESP32_RXD: now also J4.5 (Pin_5)
- net ESP32_TXD: now reaches U2.37 (TXD0/IO43)
- net ESP32_TXD: now also J4.3 (Pin_3)
- net at D18.1 (A1), U16.18 (CANL): now also J13.8 (Pin_8), J7.2 (Pin_2)
- net at D18.2 (A2), U16.19 (CANH): now also J13.7 (Pin_7), J7.4 (Pin_4)
- net at R1.1: now also C1.+; no longer C1.1
- net at D17.1 (A1), U15.18 (CANL): now also J12.8 (Pin_8), J6.2 (Pin_2)
- net at D17.2 (A2), U15.19 (CANH): now also J12.7 (Pin_7), J6.4 (Pin_4)
- net at D20.2 (A2), U18.19 (CANH): now also J15.7 (Pin_7), J9.4 (Pin_4)
- net at D20.1 (A1), U18.18 (CANL): now also J15.8 (Pin_8), J9.2 (Pin_2)
- net ~{INT_CAN2}: now reaches U9.12 (~{INT})
- net ~{INT_CAN2}: now also U2.33 (IO40)
- net CAN1-: now reaches U14.3 (TXD), U8.1 (TXCAN)
- net CAN1+: now reaches U14.5 (RXD), U8.2 (RXCAN)
- net ~{INT_CAN1}: now reaches U8.12 (~{INT})
- net ~{INT_CAN1}: now also U2.35 (IO42)
- net ~{INT_CAN5}: now reaches U12.12 (~{INT})
- net ~{INT_CAN5}: now also U2.21 (IOA13)
- net ~{RTC_RESET}: no longer names the net of U6.11 (P6)
- new net: J6.1 (Pin_1), R42.2
- new net: J6.3 (Pin_3), R41.2
- new net: U19.16 (GISOIN), U19.17 (GISOIN)
- new net: U17.16 (GISOIN), U17.17 (GISOIN)
- new net: J8.1 (Pin_1), R46.2
- new net: J8.3 (Pin_3), R45.2
- new net: TP1.1, U1.1 (CLKOUT)
- new net: R6.2, U1.8 (EVI)
- new net: D22.2 (A), R51.1
- new net: J5.1 (Pin_1), R40.2
- new net: J5.3 (Pin_3), R39.2
- new net: C94.1, R43.1, R44.1
- new net: C92.1, R39.1, R40.1
- new net: D4.C (K), U4.3 (VI)
- new net: U16.16 (GISOIN), U16.17 (GISOIN)
- new net: J7.1 (Pin_1), R44.2
- new net: J7.3 (Pin_3), R43.2
- new net: D5.C (K), U5.1 (VIN)
- new net: C97.1, R49.1, R50.1
- new net: J10.1 (Pin_1), R50.2
- new net: C96.1, R47.1, R48.1
- new net: J9.1 (Pin_1), R48.2
- new net: C95.1, R45.1, R46.1
- new net: C93.1, R41.1, R42.1
- new net: J9.3 (Pin_3), R47.2
- new net: U15.16 (GISOIN), U15.17 (GISOIN)
- new net: J10.3 (Pin_3), R49.2
- new net: D3.C (K), U3.3 (VI)
- new net: U14.16 (GISOIN), U14.17 (GISOIN)
- new net: U18.16 (GISOIN), U18.17 (GISOIN)
- new net ESP_BOOT: C5.2, J4.6 (Pin_6), SW2.2, U2.27 (IO0)
- no-connect marks 0 -> 1
Other:
- note added: "ESP32 Programming Header"
- note added: "ESP32-S3-WROOM-1U-N8R8"
- note added: "I²C Address: 0x52"
- note added: "TODO: X Add termination resistors/jumpers to CAN lines X Swap microSD socket to full SD socket X Change RJ45 pinout to VE.Can pinout X Double check SPI pinout on ESP32 X Reverse CAN ~{RST} bias so that devices are held in reset by default X Move LED off IO0 and add 0.1 capacitor X Address USB power situation X Connect CAN ~{INT} lines to ESP32 X Breakout EN, IO0, U0TXD, U0RXD, 3.3V and GND X Upda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"
- note removed: "8P8C Pin Assignments as per CAN in Automation (CiA) Technical Report CiA 106 Figure 3 and Table 5"
- note removed: "ESP32-S3-WROOM"
- note removed: "I²C Address: 0xD2"
- note removed: "TODO: -Add termination resistors/jumpers to CAN lines -Swap microSD socket to full SD socket -Change RJ45 pinout to VE.Can pinout"
- moved on the sheet: C1, C10, C2, C4, C6, C7, C8, C9, D1, D16, D17, D18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

Commit message: Layout v01
-Add Silk
-Ground Stitching
Connections:
- new net: U19.16 (GISOIN), U19.17 (GISOIN)
- new net: U17.16 (GISOIN), U17.17 (GISOIN)
- new net: U16.16 (GISOIN), U16.17 (GISOIN)
- new net: U15.16 (GISOIN), U15.17 (GISOIN)
- new net: U14.16 (GISOIN), U14.17 (GISOIN)
- new net: U18.16 (GISOIN), U18.17 (GISOIN)
Other:
- note added: "Power Indicator LEDs"
- note removed: "TODO: X Add termination resistors/jumpers to CAN lines X Swap microSD socket to full SD socket X Change RJ45 pinout to VE.Can pinout X Double check SPI pinout on ESP32 X Reverse CAN ~{RST} bias so that devices are held in reset by default X Move LED off IO0 and add 0.1 capacitor X Address USB power situation X Connect CAN ~{INT} lines to ESP32 X Breakout EN, IO0, U0TXD, U0RXD, 3.3V and GND X Upda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"
- moved on the sheet: C10, C11, C12, C13, C14, C15, C16, C4, C5, C6, C7, C9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
